Commit message: rviz urdf bringup works. fixed urdf issues. the castor wheels wobble. have choses axis in a wrong point. fix this

File: src/robot_description/urdf/AEP_Robot.urdf (robot description, URDF)
Before this commit: robot AEP_Robot, 8 links, 7 joints
Links:
- link back_castor_body_link: geometry collision mesh filename=package://robot_description/meshes/back_castor_body_link.STL; visual mesh filename=package://robot_description/meshes/back_castor_body_link.STL
- link back_castor_wheel_link: geometry collision mesh filename=package://robot_description/meshes/back_castor_wheel_link.S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; visual mesh filename=package://robot_description/meshes/back_castor_wheel_link.S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
- link base_link: geometry collision mesh filename=package://robot_description/meshes/base_link.STL; visual mesh filename=package://robot_description/meshes/base_link.STL
- link front_castor_body_link: geometry collision mesh filename=package://robot_description/meshes/front_castor_body_link.S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; visual mesh filename=package://robot_description/meshes/front_castor_body_link.S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
- link front_castor_wheel_link: geometry collision mesh filename=package://robot_description/meshes/front_castor_wheel_link.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; visual mesh filename=package://robot_description/meshes/front_castor_wheel_link.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
- link left_wheel_link: geometry collision mesh filename=package://robot_description/meshes/left_wheel_link.STL; visual mesh filename=package://robot_description/meshes/left_wheel_link.STL
- link lidar_link: geometry collision mesh filename=package://robot_description/meshes/lidar_link.STL; visual mesh filename=package://robot_description/meshes/lidar_link.STL
- link right_wheel_link: geometry collision mesh filename=package://robot_description/meshes/right_wheel_link.STL; visual mesh filename=package://robot_description/meshes/right_wheel_link.STL
Joints:
- joint back_castor_body_joint: limit lower=0 upper=0 effort=0 velocity=0 -> (none); type revolute -> continuous
- joint back_castor_wheel_joint: limit lower=0 upper=0 effort=0 velocity=0 -> (none); type revolute -> continuous
- joint front_castor_body_joint: limit lower=0 upper=0 effort=0 velocity=0 -> (none); type revolute -> continuous
- joint front_castor_wheel_joint: limit lower=0 upper=0 effort=0 velocity=0 -> (none); type revolute -> continuous
- joint left_wheel_joint: limit lower=0 upper=0 effort=0 velocity=0 -> (none); type revolute -> continuous
- joint right_wheel_joint: limit lower=0 upper=0 effort=0 velocity=0 -> (none); type revolute -> continuous
