Commit message: joint state publisher for wheels are not spawning

File: src/robot_description/urdf/AEP_Robot_macro.urdf.xacro (robot description, xacro)
@@ -7,11 +7,5 @@
         <origin xyz="-0.0023189 0.0073427 0.1843" rpy="0 0 0" />
         <mass value="15.896" />
-        <inertia
-          ixx="0.65725"
-          ixy="-3.6456E-08"
-          ixz="0.040641"
-          iyy="0.58335"
-          iyz="-2.2784E-12"
-          izz="0.1582" />
+        <inertia ixx="0.65725" ixy="-3.6456E-08" ixz="0.040641" iyy="0.58335" iyz="-2.2784E-12" izz="0.1582" />
       </inertial>
       <visual>
@@ -31,4 +25,18 @@
       </collision>
     </link>
+    <!-- Gazebo diff-drive plugin -->
+    <gazebo reference="${prefix}base_link">
+      <plugin name="gz::plugin::DiffDrive" filename="gz-sim-diff-drive-system">
+        <left_joint>${prefix}left_wheel_joint</left_joint>
+        <right_joint>${prefix}right_wheel_joint</right_joint>
+        <wheel_separation>0.5897</wheel_separation>
+        <wheel_radius>0.1</wheel_radius>
+        <odom_publish_rate>50</odom_publish_rate>
+        <topic>cmd_vel</topic>
+        <odom_topic>odom</odom_topic>
+        <odom_frame>odom</odom_frame>
+        <robot_base_frame>${prefix}base_link</robot_base_frame>
+      </plugin>
+    </gazebo>
     <!-- lidar -->
     <link name="${prefix}lidar_link">
@@ -36,11 +44,5 @@
         <origin xyz="-9.1926E-05 -0.0067665 -0.0073819" rpy="0 0 0" />
         <mass value="1.3308" />
-        <inertia
-          ixx="0.0009607"
-          ixy="8.0198E-07"
-          ixz="-3.0916E-06"
-          iyy="0.00061492"
-          iyz="-0.00015824"
-          izz="0.0010982" />
+        <inertia ixx="0.0009607" ixy="8.0198E-07" ixz="-3.0916E-06" iyy="0.00061492" iyz="-0.00015824" izz="0.0010982" />
       </inertial>
       <visual>
@@ -59,11 +61,137 @@
         </geometry>
       </collision>
+      <!-- Gazebo LiDAR sensor plugin -->
+      <gazebo reference="${prefix}lidar_link">
+        <sensor name="lidar" type="ray">
+          <pose>0 0 0 0 0 0</pose>
+          <visualize>true</visualize>
+          <update_rate>10</update_rate>
+          <ray>
+            <scan>
+              <horizontal>
+                <samples>360</samples>
+                <resolution>1.0</resolution>
+                <min_angle>-3.14159</min_angle>
+                <max_angle>3.14159</max_angle>
+              </horizontal>
+            </scan>
+            <range>
+              <min>0.12</min>
+              <max>12.0</max>
+              <resolution>0.01</resolution>
+            </range>
+            <noise>
+              <type>gaussian</type>
+              <mean>0.0</mean>
+              <stddev>0.01</stddev>
+            </noise>
+          </ray>
+          <plugin name="gz::sensors::Lidar" filename="gz-sensors-lidar">
+            <topic>scan</topic>
+            <frame_id>${prefix}lidar_link</frame_id>
+          </plugin>
+        </sensor>
+      </gazebo>
     </link>
     <joint name="${prefix}lidar_joint" type="fixed">
       <origin xyz="0 0.000420393431200835 0.32565" rpy="0 0 0" />
       <parent link="${prefix}base_link" />
-      <child  link="${prefix}lidar_link" />
+      <child link="${prefix}lidar_link" />
       <axis xyz="0 0 0" />
     </joint>
+    <!-- IMU link -->
+    <link name="${prefix}imu_link">
+      <inertial>
+        <origin xyz="0 0 0" rpy="0 0 0" />
+        <mass value="0.01" />
+        <inertia ixx="0.00001" ixy="0.0" ixz="0.0" iyy="0.00001" iyz="0.0" izz="0.00001" />
+      </inertial>
+      <visual>
+        <origin xyz="0 0 0" rpy="0 0 0" />
+        <geometry>
+          <box size="0.02 0.02 0.01" />
+        </geometry>
+        <material name="">
+          <color rgba="0 1 0 0.5" />
+        </material>
+      </visual>
+      <collision>
+        <origin xyz="0 0 0" rpy="0 0 0" />
+        <geometry>
+          <box size="0.02 0.02 0.01" />
+        </geometry>
+      </collision>
+    </link>
+    <joint name="${prefix}imu_joint" type="fixed">
+      <origin xyz="0 0 0.15" rpy="0 0 0" />
+      <parent link="${prefix}base_link" />
+      <child link="${prefix}imu_link" />
+    </joint>
+    <!-- Gazebo IMU sensor plugin -->
+    <!-- NOTE: IMU plugin temporarily commented out due to plugin loading issues -->
+    <!-- The imu_link still exists in URDF for future use -->
+    <!-- To enable IMU, uncomment below and ensure correct plugin is installed -->
+    <!--
+    <gazebo reference="${prefix}imu_link">
+      <sensor name="imu_sensor" type="imu">
+        <always_on>true</always_on>
+        <update_rate>100</update_rate>
+        <imu>
+          <angular_velocity>
+            <x>
+              <noise type="gaussian">
+                <mean>0.0</mean>
+                <stddev>0.0002</stddev>
+                <bias_mean>0.0</bias_mean>
+                <bias_stddev>0.0</bias_stddev>
+              </noise>
+            </x>
+            <y>
+              <noise type="gaussian">
+                <mean>0.0</mean>
+                <stddev>0.0002</stddev>
+                <bias_mean>0.0</bias_mean>
+                <bias_stddev>0.0</bias_stddev>
+              </noise>
+            </y>
+            <z>
+              <noise type="gaussian">
+                <mean>0.0</mean>
+                <stddev>0.0002</stddev>
+                <bias_mean>0.0</bias_mean>
+                <bias_stddev>0.0</bias_stddev>
+              </noise>
+            </z>
+          </angular_velocity>
+          <linear_acceleration>
+            <x>
+              <noise type="gaussian">
+                <mean>0.0</mean>
+                <stddev>0.017</stddev>
+                <bias_mean>0.0</bias_mean>
+                <bias_stddev>0.0</bias_stddev>
+              </noise>
+            </x>
+            <y>
+              <noise type="gaussian">
+                <mean>0.0</mean>
+                <stddev>0.017</stddev>
+                <bias_mean>0.0</bias_mean>
+                <bias_stddev>0.0</bias_stddev>
+              </noise>
+            </y>
+            <z>
+              <noise type="gaussian">
+                <mean>0.0</mean>
+                <stddev>0.017</stddev>
+                <bias_mean>0.0</bias_mean>
+                <bias_stddev>0.0</bias_stddev>
+              </noise>
+            </z>
+          </linear_acceleration>
+        </imu>
+      </sensor>
+    </gazebo>
+    -->
     <!-- left wheel -->
     <link name="${prefix}left_wheel_link">
@@ -71,11 +199,5 @@
         <origin xyz="8.211E-08 -0.017522 -4.1793E-07" rpy="0 0 0" />
         <mass value="0.583" />
-        <inertia
-          ixx="0.00092026"
-          ixy="2.1255E-10"
-          ixz="8.2654E-07"
-          iyy="0.0017198"
-          iyz="-1.099E-09"
-          izz="0.00091447" />
+        <inertia ixx="0.00092026" ixy="2.1255E-10" ixz="8.2654E-07" iyy="0.0017198" iyz="-1.099E-09" izz="0.00091447" />
       </inertial>
       <visual>
@@ -89,7 +211,7 @@
       </visual>
       <collision>
-        <origin xyz="0 0 0" rpy="0 0 0" />
-        <geometry>
-          <mesh filename="package://robot_description/meshes/left_wheel_link.STL" />
+        <origin xyz="0 0 0" rpy="1.5708 0 0" />
+        <geometry>
+          <cylinder radius="0.1" length="0.05" />
         </geometry>
       </collision>
@@ -98,7 +220,6 @@
       <origin xyz="0 0.29485 -0.025" rpy="0 0 0" />
       <parent link="${prefix}base_link" />
-      <child  link="${prefix}left_wheel_link" />
+      <child link="${prefix}left_wheel_link" />
       <axis xyz="0 1 0" />
-      <limit lower="0" upper="0" effort="0" velocity="0" />
     </joint>
     <!-- right wheel -->
@@ -107,11 +228,5 @@
         <origin xyz="3.8174E-07 0.017522 1.8833E-07" rpy="0 0 0" />
         <mass value="0.583" />
-        <inertia
-          ixx="0.00091579"
-          ixy="-1.3235E-09"
-          ixz="-2.5693E-06"
-          iyy="0.0017198"
-          iyz="-7.3676E-10"
-          izz="0.00091893" />
+        <inertia ixx="0.00091579" ixy="-1.3235E-09" ixz="-2.5693E-06" iyy="0.0017198" iyz="-7.3676E-10" izz="0.00091893" />
       </inertial>
       <visual>
@@ -125,7 +240,7 @@
       </visual>
       <collision>
-        <origin xyz="0 0 0" rpy="0 0 0" />
-        <geometry>
-          <mesh filename="package://robot_description/meshes/right_wheel_link.STL" />
+        <origin xyz="0 0 0" rpy="1.5708 0 0" />
+        <geometry>
+          <cylinder radius="0.1" length="0.05" />
         </geometry>
       </collision>
@@ -134,7 +249,6 @@
       <origin xyz="0 -0.29485 -0.025" rpy="0 0 0" />
       <parent link="${prefix}base_link" />
-      <child  link="${prefix}right_wheel_link" />
+      <child link="${prefix}right_wheel_link" />
       <axis xyz="0 1 0" />
-      <limit lower="0" upper="0" effort="0" velocity="0" />
     </joint>
     <!-- front caster -->
@@ -143,11 +257,5 @@
         <origin xyz="0.0055133 0.00033058 -0.0066169" rpy="0 0 0" />
         <mass value="0.011291" />
-        <inertia
-          ixx="4.0603E-06"
-          ixy="1.367E-08"
-          ixz="8.6782E-07"
-          iyy="3.8335E-06"
-          iyz="5.2075E-08"
-          izz="4.4634E-06" />
+        <inertia ixx="4.0603E-06" ixy="1.367E-08" ixz="8.6782E-07" iyy="3.8335E-06" iyz="5.2075E-08" izz="4.4634E-06" />
       </inertial>
       <visual>
@@ -170,7 +278,6 @@
       <origin xyz="0.105 0 -0.0415" rpy="0 0 0" />
       <parent link="${prefix}base_link" />
-      <child  link="${prefix}front_castor_body_link" />
+      <child link="${prefix}front_castor_body_link" />
       <axis xyz="0 0 1" />
-      <limit lower="0" upper="0" effort="0" velocity="0" />
     </joint>
     <link name="${prefix}front_castor_wheel_link">
@@ -178,11 +285,5 @@
         <origin xyz="0.001327 -0.02196 3.518E-06" rpy="0 0 0" />
         <mass value="0.047259" />
-        <inertia
-          ixx="9.5221E-06"
-          ixy="-2.7895E-07"
-          ixz="2.5434E-09"
-          iyy="1.4162E-05"
-          iyz="1.5234E-10"
-          izz="9.4977E-06" />
+        <inertia ixx="9.5221E-06" ixy="-2.7895E-07" ixz="2.5434E-09" iyy="1.4162E-05" iyz="1.5234E-10" izz="9.4977E-06" />
       </inertial>
       <visual>
@@ -205,7 +306,6 @@
       <origin xyz="0.021643 0.023336 -0.033" rpy="0 0 0" />
       <parent link="${prefix}front_castor_body_link" />
-      <child  link="${prefix}front_castor_wheel_link" />
+      <child link="${prefix}front_castor_wheel_link" />
       <axis xyz="0 1 0" />
-      <limit lower="0" upper="0" effort="0" velocity="0" />
     </joint>
     <!-- back caster -->
@@ -214,11 +314,5 @@
         <origin xyz="-0.0055142 -0.00031498 -0.0066169" rpy="0 0 0" />
         <mass value="0.011291" />
-        <inertia
-          ixx="4.0603E-06"
-          ixy="1.3028E-08"
-          ixz="-8.6797E-07"
-          iyy="3.8334E-06"
-          iyz="-4.9618E-08"
-          izz="4.4634E-06" />
+        <inertia ixx="4.0603E-06" ixy="1.3028E-08" ixz="-8.6797E-07" iyy="3.8334E-06" iyz="-4.9618E-08" izz="4.4634E-06" />
       </inertial>
       <visual>
@@ -241,7 +335,6 @@
       <origin xyz="-0.105 0 -0.0415" rpy="0 0 0" />
       <parent link="${prefix}base_link" />
-      <child  link="${prefix}back_castor_body_link" />
+      <child link="${prefix}back_castor_body_link" />
       <axis xyz="0 0 1" />
-      <limit lower="0" upper="0" effort="0" velocity="0" />
     </joint>
     <link name="${prefix}back_castor_wheel_link">
@@ -249,11 +342,5 @@
         <origin xyz="0.001265 -0.021964 -2.6984E-06" rpy="0 0 0" />
         <mass value="0.047259" />
-        <inertia
-          ixx="9.5208E-06"
-          ixy="-2.6579E-07"
-          ixz="-1.9877E-09"
-          iyy="1.4164E-05"
-          iyz="-1.1341E-10"
-          izz="9.4974E-06" />
+        <inertia ixx="9.5208E-06" ixy="-2.6579E-07" ixz="-1.9877E-09" iyy="1.4164E-05" iyz="-1.1341E-10" izz="9.4974E-06" />
       </inertial>
       <visual>
@@ -276,8 +363,57 @@
       <origin xyz="-0.024216 0.020654 -0.033" rpy="0 0 0" />
       <parent link="${prefix}back_castor_body_link" />
-      <child  link="${prefix}back_castor_wheel_link" />
+      <child link="${prefix}back_castor_wheel_link" />
       <axis xyz="0 1 0" />
-      <limit lower="0" upper="0" effort="0" velocity="0" />
-    </joint>
+    </joint>
+    <!-- Gazebo ROS 2 control plugin -->
+    <gazebo>
+      <plugin filename="libgz_ros2_control-system.so" name="gz_ros2_control::GazeboSimROS2ControlPlugin">
+        <parameters>/home/kiran_gunathilaka/development/ros/exam_bot_ws/src/robot_description/config/controllers.yaml</parameters>
+        <controller_manager_name>controller_manager</controller_manager_name>
+      </plugin>
+    </gazebo>
+    <!-- ros2_control hardware description -->
+    <!-- Provides joint state interfaces for all joints (wheels + casters) -->
+    <ros2_control name="GazeboSimSystem" type="system">
+      <hardware>
+        <plugin>gz_ros2_control/GazeboSimSystem</plugin>
+      </hardware>
+      <!-- Left wheel joint - state only (diff-drive plugin controls it) -->
+      <joint name="${prefix}left_wheel_joint">
+        <state_interface name="position"/>
+        <state_interface name="velocity"/>
+        <state_interface name="effort"/>
+      </joint>
+      <!-- Right wheel joint - state only (diff-drive plugin controls it) -->
+      <joint name="${prefix}right_wheel_joint">
+        <state_interface name="position"/>
+        <state_interface name="velocity"/>
+        <state_interface name="effort"/>
+      </joint>
+      <!-- Front caster body joint - state only (passive) -->
+      <joint name="${prefix}front_castor_body_joint">
+        <state_interface name="position"/>
+        <state_interface name="velocity"/>
+        <state_interface name="effort"/>
+      </joint>
+      <!-- Front caster wheel joint - state only (passive) -->
+      <joint name="${prefix}front_castor_wheel_joint">
+        <state_interface name="position"/>
+        <state_interface name="velocity"/>
+        <state_interface name="effort"/>
+      </joint>
+      <!-- Back caster body joint - state only (passive) -->
+      <joint name="${prefix}back_castor_body_joint">
+        <state_interface name="position"/>
+        <state_interface name="velocity"/>
+        <state_interface name="effort"/>
+      </joint>
+      <!-- Back caster wheel joint - state only (passive) -->
+      <joint name="${prefix}back_castor_wheel_joint">
+        <state_interface name="position"/>
+        <state_interface name="velocity"/>
+        <state_interface name="effort"/>
+      </joint>
+    </ros2_control>
   </xacro:macro>
 </robot>

File: src/robot_description/urdf/main.urdf.xacro (robot description, xacro)
@@ -1,5 +1,5 @@
 <?xml version="1.0"?>
 <robot name="AEP_Robot" xmlns:xacro="http://www.ros.org/wiki/xacro">
-  <xacro:include filename="$(find robot_description)/urdf/AEP_Robot_macro.urdf.xacro"/>
+  <xacro:include filename="AEP_Robot_macro.urdf.xacro"/>
   <xacro:AEP_Robot prefix=""/>
 </robot>

Commit message: urdf fixed, timing or some issue there. lidar topic not published

File: src/robot_description/urdf/AEP_Robot_macro.urdf.xacro (robot description, xacro)
@@ -2,4 +2,19 @@
 <robot xmlns:xacro="http://www.ros.org/wiki/xacro">
   <xacro:macro name="AEP_Robot" params="prefix:=">
+    <!-- Gazebo joint state publisher (MODEL SCOPE) -->
+    <gazebo>
+      <plugin filename="gz-sim8-joint-state-publisher-system"
+          name="gz::sim::systems::JointStatePublisher">
+        <!-- Use a clear gazebo topic name -->
+        <topic>/joint_states</topic>
+        <!-- Publish only the joints you want -->
+        <joint_name>${prefix}left_wheel_joint</joint_name>
+        <joint_name>${prefix}right_wheel_joint</joint_name>
+        <joint_name>${prefix}front_castor_body_joint</joint_name>
+        <joint_name>${prefix}front_castor_wheel_joint</joint_name>
+        <joint_name>${prefix}back_castor_body_joint</joint_name>
+        <joint_name>${prefix}back_castor_wheel_joint</joint_name>
+      </plugin>
+    </gazebo>
     <!-- base_link -->
     <link name="${prefix}base_link">
@@ -25,16 +40,19 @@
       </collision>
     </link>
-    <!-- Gazebo diff-drive plugin -->
-    <gazebo reference="${prefix}base_link">
-      <plugin name="gz::plugin::DiffDrive" filename="gz-sim-diff-drive-system">
+    <!-- Gazebo diff-drive plugin (MODEL SCOPE) -->
+    <gazebo>
+      <plugin name="gz::sim::systems::DiffDrive" filename="gz-sim8-diff-drive-system">
         <left_joint>${prefix}left_wheel_joint</left_joint>
         <right_joint>${prefix}right_wheel_joint</right_joint>
         <wheel_separation>0.5897</wheel_separation>
         <wheel_radius>0.1</wheel_radius>
-        <odom_publish_rate>50</odom_publish_rate>
-        <topic>cmd_vel</topic>
-        <odom_topic>odom</odom_topic>
-        <odom_frame>odom</odom_frame>
-        <robot_base_frame>${prefix}base_link</robot_base_frame>
+        <odom_publish_frequency>50</odom_publish_frequency>
+        <!-- cmd vel in Gazebo -->
+        <topic>/cmd_vel</topic>
+        <!-- Odometry + TF output in Gazebo -->
+        <odom_topic>/odom</odom_topic>
+        <tf_topic>/tf</tf_topic>
+        <frame_id>odom</frame_id>
+        <child_frame_id>base_link</child_frame_id>
       </plugin>
     </gazebo>
@@ -366,54 +384,4 @@
       <axis xyz="0 1 0" />
     </joint>
-    <!-- Gazebo ROS 2 control plugin -->
-    <gazebo>
-      <plugin filename="libgz_ros2_control-system.so" name="gz_ros2_control::GazeboSimROS2ControlPlugin">
-        <parameters>/home/kiran_gunathilaka/development/ros/exam_bot_ws/src/robot_description/config/controllers.yaml</parameters>
-        <controller_manager_name>controller_manager</controller_manager_name>
-      </plugin>
-    </gazebo>
-    <!-- ros2_control hardware description -->
-    <!-- Provides joint state interfaces for all joints (wheels + casters) -->
-    <ros2_control name="GazeboSimSystem" type="system">
-      <hardware>
-        <plugin>gz_ros2_control/GazeboSimSystem</plugin>
-      </hardware>
-      <!-- Left wheel joint - state only (diff-drive plugin controls it) -->
-      <joint name="${prefix}left_wheel_joint">
-        <state_interface name="position"/>
-        <state_interface name="velocity"/>
-        <state_interface name="effort"/>
-      </joint>
-      <!-- Right wheel joint - state only (diff-drive plugin controls it) -->
-      <joint name="${prefix}right_wheel_joint">
-        <state_interface name="position"/>
-        <state_interface name="velocity"/>
-        <state_interface name="effort"/>
-      </joint>
-      <!-- Front caster body joint - state only (passive) -->
-      <joint name="${prefix}front_castor_body_joint">
-        <state_interface name="position"/>
-        <state_interface name="velocity"/>
-        <state_interface name="effort"/>
-      </joint>
-      <!-- Front caster wheel joint - state only (passive) -->
-      <joint name="${prefix}front_castor_wheel_joint">
-        <state_interface name="position"/>
-        <state_interface name="velocity"/>
-        <state_interface name="effort"/>
-      </joint>
-      <!-- Back caster body joint - state only (passive) -->
-      <joint name="${prefix}back_castor_body_joint">
-        <state_interface name="position"/>
-        <state_interface name="velocity"/>
-        <state_interface name="effort"/>
-      </joint>
-      <!-- Back caster wheel joint - state only (passive) -->
-      <joint name="${prefix}back_castor_wheel_joint">
-        <state_interface name="position"/>
-        <state_interface name="velocity"/>
-        <state_interface name="effort"/>
-      </joint>
-    </ros2_control>
   </xacro:macro>
 </robot>

Commit message: now not spawning in gz

File: src/robot_description/urdf/AEP_Robot_macro.urdf.xacro (robot description, xacro)
@@ -17,4 +17,6 @@
       </plugin>
     </gazebo>
+    <!-- base_footprint (root, no inertial) -->
+    <link name="${prefix}base_footprint" />
     <!-- base_link -->
     <link name="${prefix}base_link">
@@ -40,4 +42,9 @@
       </collision>
     </link>
+    <joint name="${prefix}base_footprint_joint" type="fixed">
+      <origin xyz="0 0 0" rpy="0 0 0" />
+      <parent link="${prefix}base_footprint" />
+      <child link="${prefix}base_link" />
+    </joint>
     <!-- Gazebo diff-drive plugin (MODEL SCOPE) -->
     <gazebo>
@@ -50,9 +57,6 @@
         <!-- cmd vel in Gazebo -->
         <topic>/cmd_vel</topic>
-        <!-- Odometry + TF output in Gazebo -->
+        <!-- Odometry output in Gazebo (TF disabled; use ROS TF only) -->
         <odom_topic>/odom</odom_topic>
-        <tf_topic>/tf</tf_topic>
-        <frame_id>odom</frame_id>
-        <child_frame_id>base_link</child_frame_id>
       </plugin>
     </gazebo>
@@ -146,70 +150,4 @@
       <child link="${prefix}imu_link" />
     </joint>
-    <!-- Gazebo IMU sensor plugin -->
-    <!-- NOTE: IMU plugin temporarily commented out due to plugin loading issues -->
-    <!-- The imu_link still exists in URDF for future use -->
-    <!-- To enable IMU, uncomment below and ensure correct plugin is installed -->
-    <!--
-    <gazebo reference="${prefix}imu_link">
-      <sensor name="imu_sensor" type="imu">
-        <always_on>true</always_on>
-        <update_rate>100</update_rate>
-        <imu>
-          <angular_velocity>
-            <x>
-              <noise type="gaussian">
-                <mean>0.0</mean>
-                <stddev>0.0002</stddev>
-                <bias_mean>0.0</bias_mean>
-                <bias_stddev>0.0</bias_stddev>
-              </noise>
-            </x>
-            <y>
-              <noise type="gaussian">
-                <mean>0.0</mean>
-                <stddev>0.0002</stddev>
-                <bias_mean>0.0</bias_mean>
-                <bias_stddev>0.0</bias_stddev>
-              </noise>
-            </y>
-            <z>
-              <noise type="gaussian">
-                <mean>0.0</mean>
-                <stddev>0.0002</stddev>
-                <bias_mean>0.0</bias_mean>
-                <bias_stddev>0.0</bias_stddev>
-              </noise>
-            </z>
-          </angular_velocity>
-          <linear_acceleration>
-            <x>
-              <noise type="gaussian">
-                <mean>0.0</mean>
-                <stddev>0.017</stddev>
-                <bias_mean>0.0</bias_mean>
-                <bias_stddev>0.0</bias_stddev>
-              </noise>
-            </x>
-            <y>
-              <noise type="gaussian">
-                <mean>0.0</mean>
-                <stddev>0.017</stddev>
-                <bias_mean>0.0</bias_mean>
-                <bias_stddev>0.0</bias_stddev>
-              </noise>
-            </y>
-            <z>
-              <noise type="gaussian">
-                <mean>0.0</mean>
-                <stddev>0.017</stddev>
-                <bias_mean>0.0</bias_mean>
-                <bias_stddev>0.0</bias_stddev>
-              </noise>
-            </z>
-          </linear_acceleration>
-        </imu>
-      </sensor>
-    </gazebo>
-    -->
     <!-- left wheel -->
     <link name="${prefix}left_wheel_link">
